File: hardware/dispo-board/connectors.kicad_sch (KiCad schematic)
At the start: 26 parts, among them J1 Conn_01x03, J10 Conn_01x02, J11 Conn_01x02, J12 Conn_01x03, J13 Conn_01x03, J14 Conn_ARM_JTAG_SWD_10, J2 Conn_01x03, J3 Conn_01x03, J4 Conn_01x04, J5 USB_B_Micro, J6 Conn_01x02, J7 Conn_01x02, J8 Conn_01x02, J9 Conn_01x02

Commit message: updated footprints, pcb
Parts:
- J1, J12, J13, J2, J3: footprint MyFootprints:solder_pad_1x3_D2.00mm -> MyFootprints:solder_pad_1x03_D3.5mm
- J10, J11, J6, J7, J8, J9: footprint MyFootprints:solder_pad_1x2_D2.00mm -> MyFootprints:solder_pad_1x02_D3.5mm
- renumbered C22 to C20, C23 to C21, C24 to C22, C25 to C23
Connections:
- net DIG_IN1: no longer C21.1, C22.1, C23.1, J7.1 (Pin_1), J8.1 (Pin_1), J9.1 (Pin_1), R7.1, R8.1, R9.1
- new net DIG_IN2: C21.1, J7.1 (Pin_1), R7.1
- new net DIG_IN3: C22.1, J8.1 (Pin_1), R8.1
- new net DIG_IN4: C23.1, J9.1 (Pin_1), R9.1
Changed lines of the file:
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@@
     )
   )
-  (global_label "DIG_IN1" (shape input) (at 137.795 66.675 0) (fields_autoplaced)
+  (global_label "DIG_IN3" (shape input) (at 137.795 66.675 0) (fields_autoplaced)
     (effects (font (size 1.27 1.27)) (justify left))
     (property "Intersheetrefs" "${INTERSHEET_REFS}" (at 148.0374 66.675 0)
@@
     )
   )
-  (global_label "DIG_IN1" (shape input) (at 182.245 66.675 0) (fields_autoplaced)
+  (global_label "DIG_IN4" (shape input) (at 182.245 66.675 0) (fields_autoplaced)
     (effects (font (size 1.27 1.27)) (justify left))
     (property "Intersheetrefs" "${INTERSHEET_REFS}" (at 192.4874 66.675 0)
@@
     )
   )
-  (global_label "GND_IN" (shape input) (at 40.005 46.355 0) (fields_autoplaced)
-    (effects (font (size 1.27 1.27)) (justify left))
-    (property "Intersheetrefs" "${INTERSHEET_REFS}" (at 49.7636 46.355 0)
+  (global_label "GND" (shape input) (at 40.005 46.355 0) (fields_autoplaced)
+    (effects (font (size 1.27 1.27)) (justify left))
+    (property "Intersheetrefs" "${INTERSHEET_REFS}" (at 46.8607 46.355 0)
       (effects (font (size 1.27 1.27)) (justify left) hide)
     )
@@
     )
   )
-  (global_label "DIG_IN1" (shape input) (at 93.345 66.675 0) (fields_autoplaced)
+  (global_label "DIG_IN2" (shape input) (at 93.345 66.675 0) (fields_autoplaced)
     (effects (font (size 1.27 1.27)) (justify left))
     (property "Intersheetrefs" "${INTERSHEET_REFS}" (at 103.5874 66.675 0)
@@
       (effects (font (size 1.27 1.27)))
     )
-    (property "Footprint" "MyFootprints:solder_pad_1x2_D2.00mm" (at 26.67 92.71 0)
+    (property "Footprint" "MyFootprints:solder_pad_1x02_D3.5mm" (at 26.67 92.71 0)
       (effects (font (size 1.27 1.27)) hide)
     )
@@
       (effects (font (size 1.27 1.27)))
     )
-    (property "Footprint" "MyFootprints:solder_pad_1x3_D2.00mm" (at 93.345 28.575 0)
+    (property "Footprint" "MyFootprints:solder_pad_1x03_D3.5mm" (at 93.345 28.575 0)
       (effects (font (size 1.27 1.27)) hide)
     )
@@
       (effects (font (size 1.27 1.27)))
     )
-    (property "Footprint" "MyFootprints:solder_pad_1x2_D2.00mm" (at 115.57 66.675 0)
+    (property "Footprint" "MyFootprints:solder_pad_1x02_D3.5mm" (at 115.57 66.675 0)
       (effects (font (size 1.27 1.27)) hide)
     )
@@
       (effects (font (size 1.27 1.27)))
     )
-    (property "Footprint" "MyFootprints:solder_pad_1x2_D2.00mm" (at 63.5 92.71 0)
+    (property "Footprint" "MyFootprints:solder_pad_1x02_D3.5mm" (at 63.5 92.71 0)
       (effects (font (size 1.27 1.27)) hide)
     )
@@
   (symbol (lib_id "Device:C") (at 122.555 71.12 0) (unit 1)
     (in_bom yes) (on_board yes) (dnp no) (fields_autoplaced)
-    (property "Reference" "C24" (at 126.365 69.85 0)
+    (property "Reference" "C22" (at 126.365 69.85 0)
       (effects (font (size 1.27 1.27)) (justify left))
     )
@@
       (project "dispo-board"
         (path "/93ea4da8-8485-4fb5-a89d-c72021d94c09/b8888756-c15f-4275-bc58-daa9bb032a86"
-          (reference "C24") (unit 1)
+          (reference "C22") (unit 1)
         )
       )
@@
       (effects (font (size 1.27 1.27)))
     )
-    (property "Footprint" "MyFootprints:solder_pad_1x2_D2.00mm" (at 160.02 66.675 0)
+    (property "Footprint" "MyFootprints:solder_pad_1x02_D3.5mm" (at 160.02 66.675 0)
       (effects (font (size 1.27 1.27)) hide)
     )
@@
       (effects (font (size 1.27 1.27)))
     )
-    (property "Footprint" "MyFootprints:solder_pad_1x3_D2.00mm" (at 65.405 28.575 0)
+    (property "Footprint" "MyFootprints:solder_pad_1x03_D3.5mm" (at 65.405 28.575 0)
       (effects (font (size 1.27 1.27)) hide)
     )
@@
   (symbol (lib_id "Device:C") (at 167.005 71.12 0) (unit 1)
     (in_bom yes) (on_board yes) (dnp no) (fields_autoplaced)
-    (property "Reference" "C25" (at 170.815 69.85 0)
+    (property "Reference" "C23" (at 170.815 69.85 0)
       (effects (font (size 1.27 1.27)) (justify left))
     )
@@
       (project "dispo-board"
         (path "/93ea4da8-8485-4fb5-a89d-c72021d94c09/b8888756-c15f-4275-bc58-daa9bb032a86"
-          (reference "C25") (unit 1)
+          (reference "C23") (unit 1)
         )
       )
@@
       (effects (font (size 1.27 1.27)))
     )
-    (property "Footprint" "MyFootprints:solder_pad_1x3_D2.00mm" (at 85.09 123.19 0)
+    (property "Footprint" "MyFootprints:solder_pad_1x03_D3.5mm" (at 85.09 123.19 0)
       (effects (font (size 1.27 1.27)) hide)
     )
@@
   (symbol (lib_id "Device:C") (at 33.655 71.12 0) (unit 1)
     (in_bom yes) (on_board yes) (dnp no) (fields_autoplaced)
-    (property "Reference" "C22" (at 37.465 69.85 0)
+    (property "Reference" "C20" (at 37.465 69.85 0)
       (effects (font (size 1.27 1.27)) (justify left))
     )
@@
       (project "dispo-board"
         (path "/93ea4da8-8485-4fb5-a89d-c72021d94c09/b8888756-c15f-4275-bc58-daa9bb032a86"
-          (reference "C22") (unit 1)
+          (reference "C20") (unit 1)
         )
       )
@@
       (effects (font (size 1.27 1.27)))
     )
-    (property "Footprint" "MyFootprints:solder_pad_1x3_D2.00mm" (at 122.555 28.575 0)
+    (property "Footprint" "MyFootprints:solder_pad_1x03_D3.5mm" (at 122.555 28.575 0)
       (effects (font (size 1.27 1.27)) hide)
     )
@@
       (effects (font (size 1.27 1.27)))
     )
-    (property "Footprint" "MyFootprints:solder_pad_1x2_D2.00mm" (at 71.12 66.675 0)
+    (property "Footprint" "MyFootprints:solder_pad_1x02_D3.5mm" (at 71.12 66.675 0)
       (effects (font (size 1.27 1.27)) hide)
     )
@@
       (effects (font (size 1.27 1.27)))
     )
-    (property "Footprint" "MyFootprints:solder_pad_1x3_D2.00mm" (at 85.09 109.855 0)
+    (property "Footprint" "MyFootprints:solder_pad_1x03_D3.5mm" (at 85.09 109.855 0)
       (effects (font (size 1.27 1.27)) hide)
     )
@@
   (symbol (lib_id "Device:C") (at 78.105 71.12 0) (unit 1)
     (in_bom yes) (on_board yes) (dnp no) (fields_autoplaced)
-    (property "Reference" "C23" (at 81.915 69.85 0)
+    (property "Reference" "C21" (at 81.915 69.85 0)
       (effects (font (size 1.27 1.27)) (justify left))
     )
@@
       (project "dispo-board"
         (path "/93ea4da8-8485-4fb5-a89d-c72021d94c09/b8888756-c15f-4275-bc58-daa9bb032a86"
-          (reference "C23") (unit 1)
+          (reference "C21") (unit 1)
         )
       )
@@
       (effects (font (size 1.27 1.27)))
     )
-    (property "Footprint" "MyFootprints:solder_pad_1x2_D2.00mm" (at 26.67 66.675 0)
-      (effects (font (size 1.27 1.27)) hide)
-    )
+    (property "Footprint" "MyFootprints:solder_pad_1x02_D3.5mm" (at 26.67 66.675 0)
+      (effects (font (size 1.27 1.27)) hide)
+    )
